File: Hardware/Input Board/Rev 1.0/Input Board.kicad_pcb (KiCad board)
At the start: 2 copper layers, 100 x 100 mm, 28 parts, among them J1 PORT B, J2 PORT A, J3 PS/2 KEYBOARD, J4 6502 Bus, J5 KEYBOARD, J6 Conn_02x08_Odd_Even, U1 65C22, U2 ATmega1284-P, U3 74HC138, Y1 16 MHz

Commit message: Restore exclude from BOM
Parts:
- D1: value D_Schottky -> 1N914
- J6: value Conn_02x08_Odd_Even -> IO SELECT
- JP1: value SolderJumper_2_Bridged -> IRQ
Changed lines of the file:
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@@
 			)
 		)
-		(property "Value" "Conn_02x08_Odd_Even"
+		(property "Value" "IO SELECT"
 			(at 1.27 20.16 90)
 			(layer "F.Fab")
@@
 		)
 		(embedded_fonts no)
-		(model "${KICAD8_3DMODEL_DIR}/Capacitor_SMD.3dshapes/C_0805_2012Metric.wrl"
+		(model "${KICAD10_3DMODEL_DIR}/Capacitor_SMD.3dshapes/C_0805_2012Metric.step"
 			(offset
 				(xyz 0 0 0)
@@
 			)
 		)
-		(property "Value" "D_Schottky"
+		(property "Value" "1N914"
 			(at 3.81 2.12 90)
 			(layer "F.Fab")
@@
 			)
 		)
-		(property "Value" "SolderJumper_2_Bridged"
+		(property "Value" "IRQ"
 			(at 0 1.9 90)
 			(layer "F.Fab")
@@
 		)
 		(embedded_fonts no)
-		(model "${KICAD8_3DMODEL_DIR}/Capacitor_SMD.3dshapes/C_0805_2012Metric.wrl"
+		(model "${KICAD10_3DMODEL_DIR}/Capacitor_SMD.3dshapes/C_0805_2012Metric.step"
 			(offset
 				(xyz 0 0 0)
@@
 		)
 		(embedded_fonts no)
-		(model "${KICAD8_3DMODEL_DIR}/Capacitor_SMD.3dshapes/C_0805_2012Metric.wrl"
+		(model "${KICAD10_3DMODEL_DIR}/Capacitor_SMD.3dshapes/C_0805_2012Metric.step"
 			(offset
 				(xyz 0 0 0)
