File: Hardware/Input Board/Rev 1.0/Input Board.kicad_sch (KiCad schematic)
At the start: 21 parts, among them J1 PORT B, J2 PORT A, J3 PS/2 KEYBOARD, J4 6502 Bus, J5 KEYBOARD, J6 Conn_02x08_Odd_Even, U1 65C22, U2 ATmega1284-P, U3 74HC138, Y1 16 MHz

Commit message: Add BOMs
Parts:
- C2, C4, D1, J1, J2, J3, J5, J6, JP1, U1, U2, Y1: now in the parts list
- J4: Other (none) -> https://www.amazon.com/Female-Headers-Connector-Header-Rasp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; now in the parts list

Commit message: Finish BOM and add to README
Parts:
- D1: value D_Schottky -> 1N914; Digikey (none) -> 1N914FS-ND
- J1, J2: Digikey (none) -> 2057-BHR-12-VUA-ND; Other (none) -> https://www.amazon.com/uxcell-2-54mm-2x6-Pin-Straight-Conne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
- J3: Mouser (none) -> 806-KMDGX-6S-BS; Other (none) -> https://www.amazon.com/dp/B08GS3QL7T
- J6: value Conn_02x08_Odd_Even -> IO SELECT; Other (none) -> https://www.amazon.com/Uxcell-Double-Straight-Header-Strip/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
- JP1: value SolderJumper_2_Bridged -> IRQ; now left out of the parts list
- U1: Mouser (none) -> 955-W65C22N6TPG-14
- U2: Digikey (none) -> ATMEGA1284-PU-ND; Mouser (none) -> 556-ATMEGA1284-PU

Commit message: Restore exclude from BOM
Parts:
- C2, C4, D1, J1, J2, J4, J5, J6, U1, U2, Y1: now left out of the parts list
- J3: symbol 6502 Parts:KMDGX-6S-BS -> Connector:Mini-DIN-6; now left out of the parts list
Changed lines of the file:
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@@
 		(body_style 1)
 		(exclude_from_sim no)
-		(in_bom yes)
+		(in_bom no)
 		(on_board yes)
 		(in_pos_files yes)
@@
 		(body_style 1)
 		(exclude_from_sim no)
-		(in_bom yes)
+		(in_bom no)
 		(on_board yes)
 		(in_pos_files yes)
@@
 		(body_style 1)
 		(exclude_from_sim no)
-		(in_bom yes)
+		(in_bom no)
 		(on_board yes)
 		(in_pos_files yes)
@@
 		(body_style 1)
 		(exclude_from_sim no)
-		(in_bom yes)
+		(in_bom no)
 		(on_board yes)
 		(in_pos_files yes)
@@
 		(body_style 1)
 		(exclude_from_sim no)
-		(in_bom yes)
+		(in_bom no)
 		(on_board yes)
 		(in_pos_files yes)
@@
 		(body_style 1)
 		(exclude_from_sim no)
-		(in_bom yes)
+		(in_bom no)
 		(on_board yes)
 		(in_pos_files yes)
@@
 		(body_style 1)
 		(exclude_from_sim no)
-		(in_bom yes)
+		(in_bom no)
 		(on_board yes)
 		(in_pos_files yes)
@@
 		(body_style 1)
 		(exclude_from_sim no)
-		(in_bom yes)
+		(in_bom no)
 		(on_board yes)
 		(in_pos_files yes)
@@
 		(body_style 1)
 		(exclude_from_sim no)
-		(in_bom yes)
+		(in_bom no)
 		(on_board yes)
 		(in_pos_files yes)
@@
 	)
 	(symbol
-		(lib_id "6502 Parts:KMDGX-6S-BS")
+		(lib_id "Connector:Mini-DIN-6")
 		(at 229.87 106.68 0)
 		(unit 1)
 		(body_style 1)
 		(exclude_from_sim no)
-		(in_bom yes)
+		(in_bom no)
 		(on_board yes)
 		(in_pos_files yes)
@@
 		(body_style 1)
 		(exclude_from_sim no)
-		(in_bom yes)
+		(in_bom no)
 		(on_board yes)
 		(in_pos_files yes)
@@
 		(body_style 1)
 		(exclude_from_sim no)
-		(in_bom yes)
+		(in_bom no)
 		(on_board yes)
 		(in_pos_files yes)
