File: Hardware/Output Board/Rev 1.0/Output Board.kicad_pcb (KiCad board)
At the start: 2 copper layers, 100 x 100 mm, 32 parts, among them J1 VDD, J2 AUDIO, J6 INT Select, J7 Conn_02x08_Odd_Even, J8 6502 Bus, U1 Pico9918A, U2 6581, U3 74HC138, U4 74HC138

Commit message: Restore exclude from BOM
Parts:
- D1: value D_Schottky -> 1N914
- J7: value Conn_02x08_Odd_Even -> IO SELECT
Changed lines of the file:
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@@
 			)
 		)
-		(property "Value" "Conn_02x08_Odd_Even"
+		(property "Value" "IO SELECT"
 			(at 1.27 20.11 0)
 			(layer "F.Fab")
@@
 			)
 		)
-		(property "Value" "D_Schottky"
+		(property "Value" "1N914"
 			(at 3.81 2.12 90)
 			(layer "F.Fab")
