File: Hardware/Output Board/Rev 1.0/Output Board.kicad_sch (KiCad schematic)
At the start: 23 parts, among them J1 VDD, J2 AUDIO, J6 INT Select, J7 Conn_02x08_Odd_Even, J8 6502 Bus, U1 Pico9918A, U2 6581, U3 74HC138, U4 74HC138

Commit message: Add BOMs
Parts:
- D1, J1, J2, J6, J7, J8, U1, U2: now in the parts list

Commit message: Finish BOM and add to README
Parts:
- D1: value D_Schottky -> 1N914; Digikey (none) -> 1N914FS-ND
- J1: Digikey (none) -> 455-2247-ND
- J2: Digikey https://www.digikey.com/en/products/detail/switchcraft-inc/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 -> PJRAN1X1U02X-ND
- J6: Other (none) -> https://www.amazon.com/Straight-Breakaway-Connector-Breadbo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
- J7: value Conn_02x08_Odd_Even -> IO SELECT; Other (none) -> https://www.amazon.com/Uxcell-Double-Straight-Header-Strip/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
- J8: Other (none) -> https://www.amazon.com/Female-Headers-Connector-Header-Rasp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
- U1: Other (none) -> https://www.tindie.com/products/visrealm/pico9918-pro/
- U2: Other (none) -> https://retrocomp.cz/produkt?id=2

Commit message: Restore exclude from BOM
Parts:
- D1, J1, J2, J6, J7, J8, U1, U2: now left out of the parts list
Changed lines of the file:
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@@
 		(body_style 1)
 		(exclude_from_sim no)
-		(in_bom yes)
+		(in_bom no)
 		(on_board yes)
 		(in_pos_files yes)
@@
 		(body_style 1)
 		(exclude_from_sim no)
-		(in_bom yes)
+		(in_bom no)
 		(on_board yes)
 		(in_pos_files yes)
@@
 		(body_style 1)
 		(exclude_from_sim no)
-		(in_bom yes)
+		(in_bom no)
 		(on_board yes)
 		(in_pos_files yes)
@@
 		(body_style 1)
 		(exclude_from_sim no)
-		(in_bom yes)
+		(in_bom no)
 		(on_board yes)
 		(in_pos_files yes)
@@
 		(body_style 1)
 		(exclude_from_sim no)
-		(in_bom yes)
+		(in_bom no)
 		(on_board yes)
 		(in_pos_files yes)
@@
 		(body_style 1)
 		(exclude_from_sim no)
-		(in_bom yes)
+		(in_bom no)
 		(on_board yes)
 		(in_pos_files yes)
@@
 		(body_style 1)
 		(exclude_from_sim no)
-		(in_bom yes)
+		(in_bom no)
 		(on_board yes)
 		(in_pos_files yes)
@@
 		(body_style 1)
 		(exclude_from_sim no)
-		(in_bom yes)
+		(in_bom no)
 		(on_board yes)
 		(in_pos_files yes)
