File: Hardware/Main Board/Rev 1.0/Main Board.kicad_pcb (KiCad board)
At the start: 2 copper layers, 100 x 100 mm, 63 parts, among them J1 PWR_SW, J10 6502 Bus, J2 Conn_02x01, J3 USB_C_Receptacle_USB2.0, J4 RESET_SW, J5 Conn_02x02_Odd_Even, J6 CLOCK_ENBL_SW, J7 Conn_01x02, J8 Conn_02x05_Odd_Even, J9 6502 Card Connector, Q1 SS8050, SW1 Reset, U1 LM555xM, U2 AS6C62256, U3 AT28C256, U4 74HC00, U5 74HC00, U6 65C02, U7 74HC00, X1 OCXO-14

Commit message: Restore exclude from BOM
Parts:
- J2: value Conn_02x01 -> ROM WE
- J5: value Conn_02x02_Odd_Even -> HRDB EN
- J7: value Conn_01x02 -> 6502 EN
- J8: value Conn_02x05_Odd_Even -> EXP EN
Connections:
- J3 pad SH: (no net) -> GND

Commit message: Change pull up resistor values
Parts:
- R10, R11, R12, R13, R14: value 1k -> 10k
