File: Hardware/Main Board/Rev 1.1/Main Board.kicad_pcb (KiCad board)
At the start: 2 copper layers, 100 x 100 mm, 63 parts, among them J1 PWR_SW, J10 6502 Bus, J2 ROM WE, J3 USB_C_Receptacle_USB2.0, J4 RESET_SW, J5 HRDB EN, J6 CLOCK_ENBL_SW, J7 6502 EN, J8 EXP EN, J9 6502 Card Connector, Q1 SS8050, SW1 Reset, U1 LM555xM, U2 AS6C62256, U3 AT28C256, U4 74HC00, U5 74HC00, U6 65C02, U7 74HC00, X1 OCXO-14

Commit message: Add Main Board Rev 1.1
Parts:
- R10, R11, R12, R13, R14: value 1k -> 10k
Other:
- board text added: "© 2024 A.C. Wright Design | acwrightdesign.com | Rev 1.1"
- board text removed: "© 2024 A.C. Wright Design | acwrightdesign.com | Rev 1.0"
