File: Hardware/Main Board/Rev 1.1/Main Board.kicad_sch (KiCad schematic)
At the start: 56 parts, among them J1 PWR_SW, J10 6502 Bus, J2 ROM WE, J3 USB_C_Receptacle_USB2.0, J4 RESET_SW, J5 HRDB EN, J6 CLOCK_ENBL_SW, J7 6502 EN, J8 EXP EN, J9 6502 Card Connector, Q1 SS8050, SW1 Reset, U1 LM555xM, U2 AS6C62256, U3 AT28C256, U4 74HC00, U5 74HC00, U6 65C02, U7 74HC00, X1 OCXO-14

Commit message: Add Main Board Rev 1.1
Parts:
- R10, R11, R12, R13, R14: value 1k -> 10k; LCSC C17513 -> C2930231
Changed lines of the file:
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@@
 		(title "6502 Main Board")
 		(date "2024-06-12")
-		(rev "1.0")
+		(rev "1.1")
 		(company "A.C. Wright Design")
 	)
@@
 			)
 		)
-		(property "Value" "1k"
+		(property "Value" "10k"
 			(at 372.11 134.2136 90)
 			(show_name no)
@@
 			)
 		)
-		(property "LCSC" "C17513"
+		(property "LCSC" "C2930231"
 			(at 372.11 137.16 0)
 			(hide yes)
@@
 			)
 		)
-		(property "Value" "1k"
+		(property "Value" "10k"
 			(at 372.11 149.4536 90)
 			(show_name no)
@@
 			)
 		)
-		(property "LCSC" "C17513"
+		(property "LCSC" "C2930231"
 			(at 372.11 152.4 0)
 			(hide yes)
@@
 			)
 		)
-		(property "Value" "1k"
+		(property "Value" "10k"
 			(at 372.11 141.8336 90)
 			(show_name no)
@@
 			)
 		)
-		(property "LCSC" "C17513"
+		(property "LCSC" "C2930231"
 			(at 372.11 144.78 0)
 			(hide yes)
@@
 			)
 		)
-		(property "Value" "1k"
+		(property "Value" "10k"
 			(at 372.11 164.6936 90)
 			(show_name no)
@@
 			)
 		)
-		(property "LCSC" "C17513"
+		(property "LCSC" "C2930231"
 			(at 372.11 167.64 0)
 			(hide yes)
@@
 			)
 		)
-		(property "Value" "1k"
+		(property "Value" "10k"
 			(at 372.11 157.0736 90)
 			(show_name no)
@@
 			)
 		)
-		(property "LCSC" "C17513"
+		(property "LCSC" "C2930231"
 			(at 372.11 160.02 0)
 			(hide yes)
